File: LAN-Module-PoE-Castellated.kicad_sch (KiCad schematic)
At the start: 105 parts, among them J1 HY931147C, J10 ProtoCastellatedHeader, J11 ProtoCastellatedHeader, J12 ProtoCastellatedHeader, J13 ProtoCastellatedHeader, J14 ProtoCastellatedHeader, J15 ProtoCastellatedHeader, J16 ProtoCastellatedHeader, J17 ProtoCastellatedHeader, J18 ProtoCastellatedHeader, J19 ProtoCastellatedHeader, J2 ProtoCastellatedHeader, J20 ProtoCastellatedHeader, J21 ProtoCastellatedHeader, J22 ProtoCastellatedHeader, J23 ProtoCastellatedHeader, J24 ProtoCastellatedHeader, J25 ProtoCastellatedHeader, J26 ProtoCastellatedHeader, J27 ProtoCastellatedHeader, J28 ProtoCastellatedHeader, J29 ProtoCastellatedHeader, J3 ProtoCastellatedHeader, J4 ProtoCastellatedHeader, J5 ProtoCastellatedHeader, J6 ProtoCastellatedHeader, J7 ProtoCastellatedHeader, J8 ProtoCastellatedHeader, J9 ProtoCastellatedHeader, SW1 RESET, U1 ESP32-U4WDH, U2 Si3404, U3 LV2842XLVDDCR, U4 RTL8201F, Y1 40MHz

Commit message: HW REV: Fix stability issue
Important change required to ensure stability across different types of ethernet switches.

I had only tested this with a TP-LINK switch, but the design did not work with other switches, and the reference schematic does NOT specify that the CT/termination resistors should be tied to 3.3V. Instead they should be coupled to GND through a capacitor (of unspecified value).
Parts:
- removed R25: 0R, Resistor_SMD:R_0603_1608Metric, symbol EspGateway-rescue:R_Small_US-device-EspGateway-rescue
Connections:
- net LAN_3P3V: no longer R13.1, R14.1, R17.1, R18.1
- net MDI0_CT: now also R13.1, R14.1, R17.1, R18.1
Other:
- note added: "NOTE: CT Must NOT be connected directly to 3.3V (causes stability issues with some switches)"
Changed lines of the file:
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@@
 	)
 	(junction
-		(at 184.15 189.23)
-		(diameter 0)
-		(color 0 0 0 0)
-	)
-	(junction
 		(at 388.62 88.9)
 		(diameter 0)
@@
 	)
 	(junction
-		(at 198.12 189.23)
-		(diameter 0)
-		(color 0 0 0 0)
-	)
-	(junction
 		(at 36.83 60.96)
 		(diameter 0)
@@
 	(wire
 		(pts
-			(xy 213.36 189.23) (xy 222.25 189.23)
+			(xy 213.36 189.23) (xy 245.11 189.23)
 		)
 		(stroke
@@
 	(wire
 		(pts
-			(xy 184.15 189.23) (xy 198.12 189.23)
-		)
-		(stroke
-			(width 0)
-			(type default)
-		)
-	)
-	(wire
-		(pts
 			(xy 83.82 71.12) (xy 83.82 68.58)
 		)
@@
 		)
 	)
-	(wire
-		(pts
-			(xy 227.33 189.23) (xy 245.11 189.23)
-		)
-		(stroke
-			(width 0)
-			(type default)
-		)
-	)
 	(polyline
 		(pts
@@
 		)
 	)
+	(text "NOTE: CT Must NOT be connected directly to 3.3V\n(causes stability issues with some switches)"
+		(exclude_from_sim no)
+		(at 238.506 186.944 0)
+		(effects
+			(font
+				(size 1.27 1.27)
+			)
+		)
+	)
 	(text "PD"
 		(exclude_from_sim no)
@@
 	)
 	(label "MDI0_CT"
-		(at 242.57 189.23 180)
+		(at 245.11 193.04 270)
 		(fields_autoplaced yes)
 		(effects
@@
 					(unit 1)
 				)
-			)
-		)
-	)
-	(symbol
-		(lib_id "EspGateway-rescue:R_Small_US-device-EspGateway-rescue")
-		(at 224.79 189.23 90)
-		(mirror x)
-		(unit 1)
-		(exclude_from_sim no)
-		(in_bom yes)
-		(on_board yes)
-		(dnp no)
-		(property "Reference" "R25"
-			(at 226.06 186.69 90)
-			(effects
-				(font
-					(size 1.27 1.27)
-				)
-				(justify left)
-			)
-		)
-		(property "Value" "0R"
-			(at 226.06 191.77 90)
-			(effects
-				(font
-					(size 1.27 1.27)
-				)
-				(justify left)
-			)
-		)
-		(property "Footprint" "Resistor_SMD:R_0603_1608Metric"
-			(at 224.79 189.23 0)
-			(effects
-				(font
-					(size 1.27 1.27)
-				)
-				(hide yes)
-			)
-		)
-		(property "Datasheet" "~"
-			(at 224.79 189.23 0)
-			(effects
-				(font
-					(size 1.27 1.27)
-				)
-				(hide yes)
-			)
-		)
-		(property "Description" ""
-			(at 224.79 189.23 0)
-			(effects
-				(font
-					(size 1.27 1.27)
-				)
-				(hide yes)
-			)
-		)
-		(property "Annotation" "DNP"
-			(at 228.6 187.96 90)
-			(effects
-				(font
-					(size 1.27 1.27)
-					(bold yes)
-				)
-			)
-		)
-		(pin "1"
-		)
-		(pin "2"
-		)
-		(instances
-			(project "LAN-Module-PoE-Castellated"
-				(path "/d0fb0864-e79b-4bdc-8e8e-eed0cabe6d56"
-					(reference "R25")
-					(unit 1)
-				)
