File: LAN-Module-PoE.kicad_sch (KiCad schematic)
At the start: 105 parts, among them J1 HY931147C, J10 ProtoCastellatedHeader, J11 ProtoCastellatedHeader, J12 ProtoCastellatedHeader, J13 ProtoCastellatedHeader, J14 ProtoCastellatedHeader, J15 ProtoCastellatedHeader, J16 ProtoCastellatedHeader, J17 ProtoCastellatedHeader, J18 ProtoCastellatedHeader, J19 ProtoCastellatedHeader, J2 ProtoCastellatedHeader, J20 ProtoCastellatedHeader, J21 ProtoCastellatedHeader, J22 ProtoCastellatedHeader, J23 ProtoCastellatedHeader, J24 ProtoCastellatedHeader, J25 ProtoCastellatedHeader, J26 ProtoCastellatedHeader, J27 ProtoCastellatedHeader, J28 ProtoCastellatedHeader, J29 ProtoCastellatedHeader, J3 ProtoCastellatedHeader, J4 ProtoCastellatedHeader, J5 ProtoCastellatedHeader, J6 ProtoCastellatedHeader, J7 ProtoCastellatedHeader, J8 ProtoCastellatedHeader, J9 ProtoCastellatedHeader, SW1 RESET, U2 Si3404, U3 LV2842XLVDDCR, U4 RTL8201F, Y1 40MHz

Commit message: Rev2.1 changes
Just changing component attributes, no design changes
Parts:
- C14: value (none) -> 10u
- C18, C29: value 2.2u -> (none); footprint Capacitor_SMD:C_0805_2012Metric -> (none); Dielectric X5R -> (none); Spec (none) -> X5R
- C28, C7: value 1u -> (none); footprint Capacitor_SMD:C_0603_1608Metric -> (none); Dielectric X5R -> (none); Spec (none) -> X5R
- C4: value 1u -> (none); footprint Capacitor_SMD:C_0805_2012Metric -> (none); Dielectric X5R -> (none); Spec (none) -> X5R
- D2: value (none) -> B5819W; footprint (none) -> Diode_SMD:D_SOD-123
- R15, R16: value (none) -> 270R
- R21: value (none) -> 33k
- R22, R4: value (none) -> 510R; footprint (none) -> Resistor_SMD:R_0603_1608Metric
- R23: value (none) -> 1k; footprint (none) -> Resistor_SMD:R_0603_1608Metric
- R24: value (none) -> 8.2k; footprint (none) -> Resistor_SMD:R_0603_1608Metric
- R26: value (none) -> 33k 1%; footprint (none) -> Resistor_SMD:R_0603_1608Metric
- R27: value (none) -> 10k 1%; footprint (none) -> Resistor_SMD:R_0603_1608Metric
- U1: value (none) -> ESP32-U4WDH; footprint (none) -> Package_DFN_QFN:QFN-48-1EP_5x5mm_P0.35mm_EP3.7x3.7mm_ThermalVias
Changed lines of the file:
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@@
       (effects (font (size 1.524 1.524)))
     )
-    (property "Value" "" (id 1) (at 120.65 33.02 0)
+    (property "Value" "ESP32-U4WDH" (id 1) (at 120.65 33.02 0)
       (effects (font (size 1.524 1.524)))
     )
-    (property "Footprint" "" (id 2) (at 120.65 120.015 0)
+    (property "Footprint" "Package_DFN_QFN:QFN-48-1EP_5x5mm_P0.35mm_EP3.7x3.7mm_ThermalVias" (id 2) (at 120.65 120.015 0)
       (effects (font (size 1.524 1.524)) hide)
     )
@@
       (effects (font (size 1.27 1.27)) (justify left))
     )
-    (property "Value" "" (id 1) (at 73.66 64.77 90)
+    (property "Value" "10u" (id 1) (at 73.66 64.77 90)
       (effects (font (size 1.27 1.27)) (justify left))
     )
@@
       (effects (font (size 1.27 1.27)) (justify left))
     )
-    (property "Value" "" (id 1) (at 96.52 111.76 90)
-      (effects (font (size 1.27 1.27)) (justify left))
-    )
-    (property "Footprint" "" (id 2) (at 93.98 109.22 0)
+    (property "Value" "510R" (id 1) (at 96.52 111.76 90)
+      (effects (font (size 1.27 1.27)) (justify left))
+    )
+    (property "Footprint" "Resistor_SMD:R_0603_1608Metric" (id 2) (at 93.98 109.22 0)
       (effects (font (size 1.27 1.27)) hide)
     )
@@
       (effects (font (size 1.27 1.27)) (justify left))
     )
-    (property "Value" "2.2u" (id 1) (at 365.5568 95.3516 0)
-      (effects (font (size 1.27 1.27)) (justify left))
-    )
-    (property "Footprint" "Capacitor_SMD:C_0805_2012Metric" (id 2) (at 363.22 96.52 0)
+    (property "Value" "" (id 1) (at 365.5568 95.3516 0)
+      (effects (font (size 1.27 1.27)) (justify left))
+    )
+    (property "Footprint" "" (id 2) (at 363.22 96.52 0)
       (effects (font (size 1.27 1.27)) hide)
     )
@@
       (effects (font (size 1.27 1.27)) (justify left))
     )
-    (property "Dielectric" "X5R" (id 5) (at 365.5568 99.9744 0)
+    (property "Spec" "X5R" (id 5) (at 365.5568 99.9744 0)
       (effects (font (size 1.27 1.27)) (justify left))
     )
@@
       (effects (font (size 1.27 1.27)) (justify left))
     )
-    (property "Value" "" (id 1) (at 203.2 223.52 90)
+    (property "Value" "270R" (id 1) (at 203.2 223.52 90)
       (effects (font (size 1.27 1.27)) (justify left))
     )
@@
       (effects (font (size 1.27 1.27)) (justify left))
     )
-    (property "Value" "" (id 1) (at 203.2 228.6 90)
+    (property "Value" "270R" (id 1) (at 203.2 228.6 90)
       (effects (font (size 1.27 1.27)) (justify left))
     )
@@
       (effects (font (size 1.27 1.27)) (justify left))
     )
-    (property "Value" "" (id 1) (at 318.77 45.72 0)
-      (effects (font (size 1.27 1.27)) (justify left))
-    )
-    (property "Footprint" "" (id 2) (at 317.5 45.72 0)
+    (property "Value" "33k 1%" (id 1) (at 318.77 45.72 0)
+      (effects (font (size 1.27 1.27)) (justify left))
+    )
+    (property "Footprint" "Resistor_SMD:R_0603_1608Metric" (id 2) (at 317.5 45.72 0)
       (effects (font (size 1.27 1.27)) hide)
     )
@@
       (effects (font (size 1.27 1.27)) (justify left))
     )
-    (property "Value" "" (id 1) (at 390.525 97.79 0)
-      (effects (font (size 1.27 1.27)) (justify left))
-    )
-    (property "Footprint" "" (id 2) (at 388.62 100.33 0)
+    (property "Value" "8.2k" (id 1) (at 390.525 97.79 0)
+      (effects (font (size 1.27 1.27)) (justify left))
+    )
+    (property "Footprint" "Resistor_SMD:R_0603_1608Metric" (id 2) (at 388.62 100.33 0)
       (effects (font (size 1.27 1.27)) hide)
     )
@@
       (effects (font (size 1.27 1.27)) (justify left))
     )
-    (property "Value" "" (id 1) (at 390.525 90.805 0)
-      (effects (font (size 1.27 1.27)) (justify left))
-    )
-    (property "Footprint" "" (id 2) (at 388.62 92.71 0)
+    (property "Value" "1k" (id 1) (at 390.525 90.805 0)
+      (effects (font (size 1.27 1.27)) (justify left))
+    )
+    (property "Footprint" "Resistor_SMD:R_0603_1608Metric" (id 2) (at 388.62 92.71 0)
       (effects (font (size 1.27 1.27)) hide)
     )
@@
       (effects (font (size 1.27 1.27)) (justify left))
     )
-    (property "Value" "" (id 1) (at 96.52 109.22 90)
+    (property "Value" "510R" (id 1) (at 96.52 109.22 90)
       (effects (font (size 1.27 1.27)) (justify left) hide)
     )
-    (property "Footprint" "" (id 2) (at 93.98 106.68 0)
+    (property "Footprint" "Resistor_SMD:R_0603_1608Metric" (id 2) (at 93.98 106.68 0)
       (effects (font (size 1.27 1.27)) hide)
     )
@@
       (effects (font (size 1.27 1.27)) (justify left))
     )
-    (property "Value" "" (id 1) (at 305.435 55.88 90)
-      (effects (font (size 1.27 1.27)) (justify left))
-    )
-    (property "Footprint" "" (id 2) (at 303.53 53.34 90)
+    (property "Value" "B5819W" (id 1) (at 305.435 55.88 90)
+      (effects (font (size 1.27 1.27)) (justify left))
+    )
+    (property "Footprint" "Diode_SMD:D_SOD-123" (id 2) (at 303.53 53.34 90)
       (effects (font (size 1.27 1.27)) hide)
     )
@@
       (effects (font (size 1.27 1.27)) (justify left))
     )
-    (property "Value" "2.2u" (id 1) (at 374.4468 95.3516 0)
-      (effects (font (size 1.27 1.27)) (justify left))
-    )
-    (property "Footprint" "Capacitor_SMD:C_0805_2012Metric" (id 2) (at 372.11 96.52 0)
+    (property "Value" "" (id 1) (at 374.4468 95.3516 0)
+      (effects (font (size 1.27 1.27)) (justify left))
+    )
+    (property "Footprint" "" (id 2) (at 372.11 96.52 0)
       (effects (font (size 1.27 1.27)) hide)
     )
@@
       (effects (font (size 1.27 1.27)) (justify left))
     )
-    (property "Dielectric" "X5R" (id 5) (at 374.4468 99.9744 0)
+    (property "Spec" "X5R" (id 5) (at 374.4468 99.9744 0)
       (effects (font (size 1.27 1.27)) (justify left))
     )
@@
       (effects (font (size 1.27 1.27)) (justify left))
     )
-    (property "Value" "" (id 1) (at 320.675 124.46 0)
+    (property "Value" "33k" (id 1) (at 320.675 124.46 0)
       (effects (font (size 1.27 1.27)) (justify left))
     )
@@
       (effects (font (size 1.27 1.27)) (justify left))
     )
-    (property "Value" "" (id 1) (at 318.77 52.07 0)
-      (effects (font (size 1.27 1.27)) (justify left))
-    )
-    (property "Footprint" "" (id 2) (at 317.5 53.34 0)
+    (property "Value" "10k 1%" (id 1) (at 318.77 52.07 0)
+      (effects (font (size 1.27 1.27)) (justify left))
+    )
+    (property "Footprint" "Resistor_SMD:R_0603_1608Metric" (id 2) (at 317.5 53.34 0)
       (effects (font (size 1.27 1.27)) hide)
     )
@@
       (effects (font (size 1.27 1.27)) (justify left))
     )
-    (property "Value" "1u" (id 1) (at 333.8068 95.3516 0)
-      (effects (font (size 1.27 1.27)) (justify left))
-    )
-    (property "Footprint" "Capacitor_SMD:C_0603_1608Metric" (id 2) (at 331.47 96.52 0)
+    (property "Value" "" (id 1) (at 333.8068 95.3516 0)
+      (effects (font (size 1.27 1.27)) (justify left))
+    )
+    (property "Footprint" "" (id 2) (at 331.47 96.52 0)
       (effects (font (size 1.27 1.27)) hide)
     )
@@
       (effects (font (size 1.27 1.27)) (justify right))
     )
-    (property "Dielectric" "X5R" (id 5) (at 333.8068 99.9744 0)
+    (property "Spec" "X5R" (id 5) (at 333.8068 99.9744 0)
       (effects (font (size 1.27 1.27)) (justify left))
     )
@@
       (effects (font (size 1.27 1.27)) (justify left))
     )
-    (property "Value" "1u" (id 1) (at 341.4268 95.3516 0)
-      (effects (font (size 1.27 1.27)) (justify left))
-    )
-    (property "Footprint" "Capacitor_SMD:C_0603_1608Metric" (id 2) (at 339.09 96.52 0)
+    (property "Value" "" (id 1) (at 341.4268 95.3516 0)
+      (effects (font (size 1.27 1.27)) (justify left))
+    )
+    (property "Footprint" "" (id 2) (at 339.09 96.52 0)
       (effects (font (size 1.27 1.27)) hide)
     )
@@
       (effects (font (size 1.27 1.27)) (justify left))
     )
-    (property "Dielectric" "X5R" (id 5) (at 341.4268 99.9744 0)
+    (property "Spec" "X5R" (id 5) (at 341.4268 99.9744 0)
       (effects (font (size 1.27 1.27)) (justify left))
     )
@@
       (effects (font (size 1.27 1.27)) (justify left))
     )
-    (property "Value" "1u" (id 1) (at 324.9168 95.3516 0)
-      (effects (font (size 1.27 1.27)) (justify left))
-    )
-    (property "Footprint" "Capacitor_SMD:C_0805_2012Metric" (id 2) (at 322.58 96.52 0)
+    (property "Value" "" (id 1) (at 324.9168 95.3516 0)
+      (effects (font (size 1.27 1.27)) (justify left))
+    )
+    (property "Footprint" "" (id 2) (at 322.58 96.52 0)
       (effects (font (size 1.27 1.27)) hide)
     )
@@
       (effects (font (size 1.27 1.27)) (justify left))
     )
-    (property "Dielectric" "X5R" (id 5) (at 324.9168 99.9744 0)
-      (effects (font (size 1.27 1.27)) (justify left))
-    )
+    (property "Spec" "X5R" (id 5) (at 324.9168 99.9744 0)
+      (effects (font (size 1.27 1.27)) (justify left))
+    )

Commit message: HW REV: Fix stability issue
Important change required to ensure stability across different types of ethernet switches.

I had only tested this with a TP-LINK switch, but the design did not work with other switches, and the reference schematic does NOT specify that the CT/termination resistors should be tied to 3.3V. Instead they should be coupled to GND through a capacitor (of unspecified value).
Parts:
- removed R25: 0R, Resistor_SMD:R_0603_1608Metric, symbol EspGateway-rescue:R_Small_US-device-EspGateway-rescue
- C18, C29: value (none) -> 2.2u; footprint (none) -> Capacitor_SMD:C_0805_2012Metric
- C28, C7: value (none) -> 1u; footprint (none) -> Capacitor_SMD:C_0603_1608Metric
- C4: value (none) -> 1u; footprint (none) -> Capacitor_SMD:C_0805_2012Metric
- J1: footprint Connector_RJ:RJ45_Wuerth_7499111446_Horizontal -> Connector_RJ:RJ45_Wuerth_7499111446_Horizontal; Part (none) -> LCSC:C12074
Connections:
- net LAN_3P3V: no longer R13.1, R14.1, R17.1, R18.1
- net MDI0_CT: now also R13.1, R14.1, R17.1, R18.1
Other:
- note added: "NOTE: CT Must NOT be connected directly to 3.3V (causes stability issues with some switches)"
- moved on the sheet: L3
