File: LAN-Module.kicad_sch (KiCad schematic)
At the start: 71 parts, among them J1 USB_B_Micro, J2 HR911105A, J3 Conn_Left, J4 ANT, J5 Conn_Right, Q1 2N7002, Q2 2N7002, SW1 RESET, U1 ESP32-U4WDH, U2 W25Q32, U3 LV2842XLVDDCR, U4 RTL8201F, U5 CP2102N-Axx-xQFN24, Y1 40MHz ±10ppm

Commit message: Layout PCB
Parts:
- J1: value USB_B_Micro -> (none); footprint Visclib:USB-B-MICRO-SMD -> (none)
- J3: value Conn_Left -> (none); footprint Connector_PinHeader_2.54mm:PinHeader_1x16_P2.54mm_Vertical -> (none)
- J5: value Conn_Right -> (none); footprint Connector_PinHeader_2.54mm:PinHeader_1x16_P2.54mm_Vertical -> (none)
- LOGO1: value (none) -> Logo; footprint (none) -> Visclib:wolfpaw-0.3
- U1: value ESP32-U4WDH -> (none); footprint Package_DFN_QFN:QFN-48-1EP_6x6mm_P0.4mm_EP4.3x4.3mm -> (none)
Connections:
- net BOOT: now also J5.5 (Pin_5); no longer J3.5 (Pin_5)
- net EN: now also J5.2 (Pin_2); no longer J3.4 (Pin_4)
- net GND: now also J5.15 (Pin_15); no longer J5.16 (Pin_16)
- net IO12: now also J3.3 (Pin_3); no longer J5.5 (Pin_5)
- net IO13: now also J3.6 (Pin_6); no longer J5.4 (Pin_4)
- net IO14: now also J3.4 (Pin_4); no longer J5.3 (Pin_3)
- net IO15: now also J3.7 (Pin_7); no longer J5.2 (Pin_2)
- net IO16: now also J3.2 (Pin_2); no longer J5.6 (Pin_6)
- net IO2: now also J3.9 (Pin_9); no longer J5.9 (Pin_9)
- net IO32: now also J5.7 (Pin_7); no longer J3.6 (Pin_6)
- net IO33: now also J5.6 (Pin_6); no longer J3.7 (Pin_7)
- net IO34: now also J5.9 (Pin_9); no longer J3.8 (Pin_8)
- net IO35: now also J5.8 (Pin_8); no longer J3.9 (Pin_9)
- net IO37: now also J5.12 (Pin_12)
- net IO38: now also J5.11 (Pin_11)
- net IO4: now also J3.8 (Pin_8); no longer J5.8 (Pin_8)
- net IO5: now also J3.10 (Pin_10); no longer J5.7 (Pin_7)
- net S_VN: now also J5.10 (Pin_10)
- net S_VP: now also J5.13 (Pin_13)
- net U0RXD: now also J5.4 (Pin_4); no longer J3.3 (Pin_3)
- net U0TXD: now also J5.3 (Pin_3); no longer J3.2 (Pin_2)
- net VIN: now also J5.16 (Pin_16); no longer J3.10 (Pin_10)
Changed lines of the file:
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@@
     (effects (font (size 1.27 1.27)) (justify left bottom))
   )
-  (text "(48V Max)" (at 341.63 207.01 0)
+  (text "(48V Max)" (at 355.6 209.55 0)
     (effects (font (size 1.27 1.27)) (justify left bottom))
   )
@@
     (effects (font (size 1.27 1.27)) (justify right bottom))
   )
+  (label "S_VN" (at 381 207.01 180)
+    (effects (font (size 1.27 1.27)) (justify right bottom))
+  )
   (label "ETH_RXD1" (at 76.2 207.01 0)
     (effects (font (size 1.27 1.27)) (justify left bottom))
@@
     (effects (font (size 1.27 1.27)) (justify left bottom))
   )
-  (label "IO12" (at 381 194.31 180)
-    (effects (font (size 1.27 1.27)) (justify right bottom))
+  (label "IO12" (at 337.82 189.23 0)
+    (effects (font (size 1.27 1.27)) (justify left bottom))
   )
   (label "DVDD10" (at 149.86 195.58 180)
@@
     (effects (font (size 1.27 1.27)) (justify right bottom))
   )
-  (label "GND" (at 381 222.25 180)
+  (label "GND" (at 381 219.71 180)
     (effects (font (size 1.27 1.27)) (justify right bottom))
   )
@@
     (effects (font (size 1.27 1.27)) (justify right bottom))
   )
-  (label "IO35" (at 337.82 204.47 0)
-    (effects (font (size 1.27 1.27)) (justify left bottom))
+  (label "IO35" (at 381 201.93 180)
+    (effects (font (size 1.27 1.27)) (justify right bottom))
   )
   (label "MDI0_P" (at 337.82 217.17 0)
     (effects (font (size 1.27 1.27)) (justify left bottom))
   )
-  (label "U0RXD" (at 337.82 189.23 0)
-    (effects (font (size 1.27 1.27)) (justify left bottom))
-  )
-  (label "EN" (at 337.82 191.77 0)
-    (effects (font (size 1.27 1.27)) (justify left bottom))
+  (label "U0RXD" (at 381 191.77 180)
+    (effects (font (size 1.27 1.27)) (justify right bottom))
+  )
+  (label "EN" (at 381 186.69 180)
+    (effects (font (size 1.27 1.27)) (justify right bottom))
   )
   (label "IO12" (at 147.32 54.61 180)
@@
     (effects (font (size 1.27 1.27)) (justify right bottom))
   )
+  (label "IO38" (at 381 209.55 180)
+    (effects (font (size 1.27 1.27)) (justify right bottom))
+  )
   (label "LAN_3P3V" (at 146.05 189.23 0)
     (effects (font (size 1.27 1.27)) (justify left bottom))
@@
     (effects (font (size 1.27 1.27)) (justify left bottom))
   )
-  (label "IO33" (at 337.82 199.39 0)
-    (effects (font (size 1.27 1.27)) (justify left bottom))
+  (label "IO33" (at 381 196.85 180)
+    (effects (font (size 1.27 1.27)) (justify right bottom))
   )
   (label "IO38" (at 99.06 69.85 180)
@@
     (effects (font (size 1.27 1.27)) (justify right bottom))
   )
+  (label "S_VP" (at 381 214.63 180)
+    (effects (font (size 1.27 1.27)) (justify right bottom))
+  )
   (label "GND" (at 337.82 184.15 0)
     (effects (font (size 1.27 1.27)) (justify left bottom))
   )
-  (label "IO13" (at 381 191.77 180)
-    (effects (font (size 1.27 1.27)) (justify right bottom))
+  (label "IO13" (at 337.82 196.85 0)
+    (effects (font (size 1.27 1.27)) (justify left bottom))
   )
   (label "SDD2" (at 133.35 142.24 0)
@@
     (effects (font (size 1.27 1.27)) (justify right bottom))
   )
-  (label "IO15" (at 381 186.69 180)
-    (effects (font (size 1.27 1.27)) (justify right bottom))
+  (label "IO15" (at 337.82 199.39 0)
+    (effects (font (size 1.27 1.27)) (justify left bottom))
   )
   (label "IO16" (at 156.21 74.93 180)
@@
     (effects (font (size 1.27 1.27)) (justify left bottom))
   )
-  (label "IO2" (at 381 204.47 180)
-    (effects (font (size 1.27 1.27)) (justify right bottom))
-  )
-  (label "IO4" (at 381 201.93 180)
-    (effects (font (size 1.27 1.27)) (justify right bottom))
+  (label "IO2" (at 337.82 204.47 0)
+    (effects (font (size 1.27 1.27)) (justify left bottom))
+  )
+  (label "IO4" (at 337.82 201.93 0)
+    (effects (font (size 1.27 1.27)) (justify left bottom))
   )
   (label "ETH_LED0" (at 219.71 226.06 180)
@@
     (effects (font (size 1.27 1.27)) (justify left bottom))
   )
+  (label "IO37" (at 381 212.09 180)
+    (effects (font (size 1.27 1.27)) (justify right bottom))
+  )
   (label "EN" (at 372.11 102.87 180)
     (effects (font (size 1.27 1.27)) (justify right bottom))
   )
-  (label "IO14" (at 381 189.23 180)
-    (effects (font (size 1.27 1.27)) (justify right bottom))
-  )
-  (label "IO32" (at 337.82 196.85 0)
-    (effects (font (size 1.27 1.27)) (justify left bottom))
+  (label "IO14" (at 337.82 191.77 0)
+    (effects (font (size 1.27 1.27)) (justify left bottom))
+  )
+  (label "IO32" (at 381 199.39 180)
+    (effects (font (size 1.27 1.27)) (justify right bottom))
   )
   (label "BOOT" (at 156.21 64.77 180)
@@
     (effects (font (size 1.27 1.27)) (justify left bottom))
   )
-  (label "IO5" (at 381 199.39 180)
-    (effects (font (size 1.27 1.27)) (justify right bottom))
-  )
-  (label "IO34" (at 337.82 201.93 0)
-    (effects (font (size 1.27 1.27)) (justify left bottom))
+  (label "IO5" (at 337.82 207.01 0)
+    (effects (font (size 1.27 1.27)) (justify left bottom))
+  )
+  (label "IO34" (at 381 204.47 180)
+    (effects (font (size 1.27 1.27)) (justify right bottom))
   )
   (label "U0RXD" (at 83.82 106.68 0)
@@
     (effects (font (size 1.27 1.27)) (justify left bottom))
   )
-  (label "IO16" (at 381 196.85 180)
-    (effects (font (size 1.27 1.27)) (justify right bottom))
+  (label "IO16" (at 337.82 186.69 0)
+    (effects (font (size 1.27 1.27)) (justify left bottom))
   )
   (label "IO15" (at 147.32 59.69 180)
     (effects (font (size 1.27 1.27)) (justify right bottom))
   )
-  (label "BOOT" (at 337.82 194.31 0)
-    (effects (font (size 1.27 1.27)) (justify left bottom))
+  (label "BOOT" (at 381 194.31 180)
+    (effects (font (size 1.27 1.27)) (justify right bottom))
   )
   (label "IO32" (at 99.06 90.17 180)
@@
     (effects (font (size 1.27 1.27)) (justify right bottom))
   )
-  (label "VIN" (at 337.82 207.01 0)
-    (effects (font (size 1.27 1.27)) (justify left bottom))
+  (label "VIN" (at 381 222.25 180)
+    (effects (font (size 1.27 1.27)) (justify right bottom))
   )
   (label "ETH_CLK" (at 76.2 256.54 0)
@@
     (effects (font (size 1.27 1.27)) (justify left bottom))
   )
-  (label "U0TXD" (at 337.82 186.69 0)
-    (effects (font (size 1.27 1.27)) (justify left bottom))
+  (label "U0TXD" (at 381 189.23 180)
+    (effects (font (size 1.27 1.27)) (justify right bottom))
   )
   (hierarchical_label "VDD" (shape input) (at 184.15 172.72 90)
@@
       (effects (font (size 1.524 1.524)))
     )
-    (property "Value" "ESP32-U4WDH" (id 1) (at 120.65 34.7726 0)
+    (property "Value" "" (id 1) (at 120.65 34.7726 0)
       (effects (font (size 1.524 1.524)))
     )
-    (property "Footprint" "Package_DFN_QFN:QFN-48-1EP_6x6mm_P0.4mm_EP4.3x4.3mm" (id 2) (at 120.65 120.015 0)
+    (property "Footprint" "" (id 2) (at 120.65 120.015 0)
       (effects (font (size 1.524 1.524)) hide)
     )
@@
     (in_bom yes) (on_board yes)
     (property "Reference" "J3" (id 0) (at 335.4832 179.451 0))
-    (property "Value" "Conn_Left" (id 1) (at 335.4832 181.7624 0))
-    (property "Footprint" "Connector_PinHeader_2.54mm:PinHeader_1x16_P2.54mm_Vertical" (id 2) (at 332.74 201.93 0)
+    (property "Value" "" (id 1) (at 335.4832 181.7624 0))
+    (property "Footprint" "" (id 2) (at 332.74 201.93 0)
       (effects (font (size 1.27 1.27)) hide)
     )
@@
     (in_bom yes) (on_board yes)
     (property "Reference" "J5" (id 0) (at 383.3368 227.965 0))
-    (property "Value" "Conn_Right" (id 1) (at 383.3368 225.6536 0))
-    (property "Footprint" "Connector_PinHeader_2.54mm:PinHeader_1x16_P2.54mm_Vertical" (id 2) (at 386.08 201.93 0)
+    (property "Value" "" (id 1) (at 383.3368 225.6536 0))
+    (property "Footprint" "" (id 2) (at 386.08 201.93 0)
       (effects (font (size 1.27 1.27)) hide)
     )
@@
       (effects (font (size 1.524 1.524)) (justify left))
     )
-    (property "Value" "" (id 1) (at 383.54 264.16 0)
+    (property "Value" "Logo" (id 1) (at 383.54 264.16 0)
       (effects (font (size 1.524 1.524)) (justify left))
     )
-    (property "Footprint" "" (id 2) (at 377.19 261.62 0)
+    (property "Footprint" "Visclib:wolfpaw-0.3" (id 2) (at 377.19 261.62 0)
       (effects (font (size 1.524 1.524)) hide)
     )
@@
     (in_bom yes) (on_board yes) (fields_autoplaced)
     (property "Reference" "J1" (id 0) (at 278.13 96.52 0))
-    (property "Value" "USB_B_Micro" (id 1) (at 278.13 99.06 0))
-    (property "Footprint" "Visclib:USB-B-MICRO-SMD" (id 2) (at 281.94 110.49 0)
+    (property "Value" "" (id 1) (at 278.13 99.06 0))
+    (property "Footprint" "" (id 2) (at 281.94 110.49 0)
       (effects (font (size 1.27 1.27)) hide)
     )
@@
     )
     (path "/eb48074c-efc6-4294-b779-3904695ef27d"
-      (reference "J1") (unit 1) (value "USB_B_Micro") (footprint "Visclib:USB-B-MICRO-SMD")
+      (reference "J1") (unit 1) (value "USB_B_Micro") (footprint "Connector_USB:USB_Micro-B_Molex_47346-0001")
     )
     (path "/46fd813e-6fbb-4d2c-9d12-43ea2e9e6362"
@@
     )
     (path "/00000000-0000-0000-0000-0000615880d5"
-      (reference "J3") (unit 1) (value "Conn_Left") (footprint "Connector_PinHeader_2.54mm:PinHeader_1x16_P2.54mm_Vertical")
+      (reference "J3") (unit 1) (value "Conn_Left") (footprint "Visclib:ProtoCastellatedHeader_1x16")
     )
     (path "/5a40e32e-7f64-4ccd-b439-e8bf37f8771b"
@@
     )
     (path "/00000000-0000-0000-0000-000061589394"
-      (reference "J5") (unit 1) (value "Conn_Right") (footprint "Connector_PinHeader_2.54mm:PinHeader_1x16_P2.54mm_Vertical")
+      (reference "J5") (unit 1) (value "Conn_Right") (footprint "Visclib:ProtoCastellatedHeader_1x16")
     )
     (path "/86bf1549-6e79-4a48-82f0-4f0a5849ddb8"
@@
     )
     (path "/00000000-0000-0000-0000-0000613daa80"
-      (reference "U1") (unit 1) (value "ESP32-U4WDH") (footprint "Package_DFN_QFN:QFN-48-1EP_6x6mm_P0.4mm_EP4.3x4.3mm")
+      (reference "U1") (unit 1) (value "ESP32-U4WDH") (footprint "Visclib:ESP32-REDUCED")
     )
     (path "/05d8c053-4ffb-44b3-92bf-c423664a709a"

Commit message: Final routing and placement
Parts:
- removed C4: 1u, Capacitor_SMD:C_0603_1608Metric, symbol EspGateway-rescue:C_Small-device-EspGateway-rescue
- removed C6: 10u, Capacitor_SMD:C_0603_1608Metric, symbol EspGateway-rescue:C_Small-device-EspGateway-rescue
- removed J3, J5: (no value), symbol Connector:Conn_01x16_Female
- removed J4: ANT, Connector_Coaxial:U.FL_Hirose_U.FL-R-SMT-1_Vertical, symbol Connector:Conn_Coaxial
- added F1: 1A, Fuse:Fuse_1206_3216Metric, symbol Device:Polyfuse_Small
- added J10, J11, J12, J13, J14, J15, J16, J17, J18, J19, J20, J21, J22, J23, J24, J25, J26, J27, J28, J3, J4, J5, J6, J7, J8, J9: ProtoCastellatedHeader, Visclib:ProtoCastellatedHeader_65mil, symbol Visclib:ProtoCastellatedHeader
- J1: value (none) -> USB_B_Micro; footprint (none) -> Connector_USB:USB_Micro-B_Molex_47346-0001
- U1: value (none) -> ESP32-U4WDH; footprint (none) -> Visclib:ESP32-REDUCED
Connections:
- net +3V3: now also L3.1, R10.1, R9.1
- net 3V3: now also J15.1
- net BOOT: now also J5.1
- net EN: now also J4.1
- net GND: now also J14.1, J16.1, J27.1, J3.1
- net IO12: now also J9.1
- net IO13: now also J6.1
- net IO14: now also J12.1
- net IO15: now also J8.1
- net IO16: now also J7.1
- net IO2: now also J11.1
- net IO32: now also J20.1
- net IO33: now also J19.1
- net IO34: now also J22.1
- net IO35: now also J21.1
- net IO37: now also J25.1
- net IO38: now also J24.1
- net IO4: now also J10.1
- net IO5: now also J13.1
- net S_VN: now also J23.1
- net S_VP: now also J26.1
- net U0RXD: now also J18.1
- net U0TXD: now also J17.1
- net VIN: now also D2.1 (K), F1.1, J28.1
- net SW: now reaches C20.2, D1.1 (K), L2.1, U3.6 (SW)
- net FB: now reaches R6.2, R7.1, U3.3 (FB)
- net RTS: now reaches Q1.1 (G), Q2.2 (S), U5.19 (~{RTS})
- net DTR: now reaches Q1.3 (D), Q2.1 (G), U5.23 (~{DTR})
- net USB_P: now reaches J1.3 (D+), U5.3 (D+)
- net USB_N: now reaches J1.2 (D-), U5.4 (D-)
- net VDD: no longer names the net of C17.1, C18.1, U3.4 (~{SHDN}), U3.5 (VIN)
- net VDD: now also F1.2; no longer D2.1 (K), L3.1, R10.1, R9.1
- no-connect marks 19 -> 20
Other:
- note added: "(40V Max)"
- note added: "VBreakdown > 40V"
- note removed: "(48V Max)"
- moved on the sheet: C11, C2, C5, D2

Commit message: Address TODOs
Parts:
- D1: value FM240W -> (none); footprint Diode_SMD:D_SOD-123 -> (none)
- D2: value FM240W -> (none)
Other:
- note added: "Ceramic caps should be X5R or X7R Diode should be fast recovery type f_sw = 550kHz"
- note added: "PHYADDR=00"
- note removed: "Ceramic caps should be X5R or X7R"
- note removed: "TODO: Confirm diode footprints"
- note removed: "TODO: Verify LED colours"
Changed lines of the file:
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@@
     (effects (font (size 1.27 1.27)) (justify left bottom))
   )
-  (text "NRS6045T6R3MMGK ??" (at 346.71 39.37 0)
+  (text "NRS6045T6R3MMGK ??" (at 345.44 38.1 0)
     (effects (font (size 1.27 1.27)) (justify left bottom))
   )
@@
   )
   (text "WiFi not used." (at 133.35 34.29 0)
-    (effects (font (size 1.27 1.27)) (justify left bottom))
-  )
-  (text "TODO: Confirm diode footprints" (at 316.23 26.67 0)
-    (effects (font (size 1.27 1.27)) (justify left bottom))
-  )
-  (text "TODO: Verify LED colours" (at 222.25 228.6 0)
     (effects (font (size 1.27 1.27)) (justify left bottom))
   )
@@
     (effects (font (size 1.27 1.27)) (justify left bottom))
   )
-  (text "Ceramic caps should be X5R or X7R" (at 302.26 60.96 0)
+  (text "Ceramic caps should be X5R or X7R\nDiode should be fast recovery type\nf_sw = 550kHz"
+    (at 302.26 64.77 0)
     (effects (font (size 1.27 1.27)) (justify left bottom))
   )
@@
     (effects (font (size 1.27 1.27)) (justify right bottom))
   )
-  (text "NOTE: Pin-compatible with LMR16006" (at 326.39 34.29 0)
+  (text "NOTE: Pin-compatible with LMR16006" (at 307.34 29.21 0)
     (effects (font (size 1.27 1.27)) (justify left bottom))
   )
@@
   )
   (text "PU" (at 149.86 59.69 0)
+    (effects (font (size 1.27 1.27)) (justify left bottom))
+  )
+  (text "PHYADDR=00" (at 195.58 240.03 0)
     (effects (font (size 1.27 1.27)) (justify left bottom))
   )
@@
       (effects (font (size 1.27 1.27)) (justify left))
     )
-    (property "Value" "FM240W" (id 1) (at 331.9272 54.483 90)
-      (effects (font (size 1.27 1.27)) (justify left))
-    )
-    (property "Footprint" "Diode_SMD:D_SOD-123" (id 2) (at 330.2 53.34 90)
+    (property "Value" "" (id 1) (at 331.9272 54.483 90)
+      (effects (font (size 1.27 1.27)) (justify left))
+    )
+    (property "Footprint" "" (id 2) (at 330.2 53.34 90)
       (effects (font (size 1.27 1.27)) hide)
     )
@@
       (effects (font (size 1.27 1.27)) (justify left))
     )
-    (property "Value" "FM240W" (id 1) (at 266.827 39.8272 90)
+    (property "Value" "" (id 1) (at 266.827 39.8272 90)
       (effects (font (size 1.27 1.27)) (justify left))
     )
@@
     )
     (path "/00000000-0000-0000-0000-0000613dac4f"
-      (reference "D1") (unit 1) (value "FM240W") (footprint "Diode_SMD:D_SOD-123")
+      (reference "D1") (unit 1) (value "PMEG6020ER,115") (footprint "Diode_SMD:D_SOD-123")
     )
     (path "/bb610d98-5315-4341-9748-5fe02e1c0831"
-      (reference "D2") (unit 1) (value "FM240W") (footprint "Diode_SMD:D_SOD-123")
+      (reference "D2") (unit 1) (value "?") (footprint "Diode_SMD:D_SOD-123")
     )
     (path "/72a5b144-a5ee-45ac-a3c7-824926b9d259"
